File: Design2_TwoBoardPogoPin/Board1 - Pad and Pogo Pin/Board1_Pad_PogoPin.kicad_sch (KiCad schematic)
At the start: 128 parts, among them J1 Conn_01x01_Pin, J10 Conn_01x01_Pin, J11 Conn_01x01_Pin, J12 Conn_01x01_Pin, J13 Conn_01x01_Pin, J14 Conn_01x01_Pin, J15 Conn_01x01_Pin, J16 Conn_01x01_Pin, J17 Conn_01x01_Pin, J18 Conn_01x01_Pin, J19 Conn_01x01_Pin, J2 Conn_01x01_Pin, J20 Conn_01x01_Pin, J21 Conn_01x01_Pin, J22 Conn_01x01_Pin, J23 Conn_01x01_Pin, J24 Conn_01x01_Pin, J25 Conn_01x01_Pin, J26 Conn_01x01_Pin, J27 Conn_01x01_Pin, J28 Conn_01x01_Pin, J29 Conn_01x01_Pin, J3 Conn_01x01_Pin, J30 Conn_01x01_Pin, J31 Conn_01x01_Pin, J32 Conn_01x01_Pin, J33 Conn_01x01_Pin, J34 Conn_01x01_Pin, J35 Conn_01x01_Pin, J36 Conn_01x01_Pin, J37 Conn_01x01_Pin, J38 Conn_01x01_Pin, J39 Conn_01x01_Pin, J4 Conn_01x01_Pin, J40 Conn_01x01_Pin, J41 Conn_01x01_Pin, J42 Conn_01x01_Pin, J43 Conn_01x01_Pin, J44 Conn_01x01_Pin, J45 Conn_01x01_Pin, J46 Conn_01x01_Pin, J47 Conn_01x01_Pin, J48 Conn_01x01_Pin, J49 Conn_01x01_Pin, J5 Conn_01x01_Pin, J50 Conn_01x01_Pin, J51 Conn_01x01_Pin, J52 Conn_01x01_Pin, J53 Conn_01x01_Pin, J54 Conn_01x01_Pin, J55 Conn_01x01_Pin, J56 Conn_01x01_Pin, J57 Conn_01x01_Pin, J58 Conn_01x01_Pin, J59 Conn_01x01_Pin, J6 Conn_01x01_Pin, J60 Conn_01x01_Pin, J61 Conn_01x01_Pin, J62 Conn_01x01_Pin, J63 Conn_01x01_Pin, J64 Conn_01x01_Pin, J7 Conn_01x01_Pin, J8 Conn_01x01_Pin, J9 Conn_01x01_Pin, U1 anode_pad, U10 anode_pad, U11 anode_pad, U12 anode_pad, U13 anode_pad, U14 anode_pad, U15 anode_pad, U16 anode_pad, U17 anode_pad, U18 anode_pad, U19 anode_pad, U2 anode_pad, U20 anode_pad, U21 anode_pad, U22 anode_pad, U23 anode_pad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

Commit message: two boards finished
Parts:
- U1, U10, U11, U12, U13, U14, U15, U16, U17, U18, U19, U2, U20, U21, U22, U23, U24, U25, U26, U27, U28, U29, U3, U30, U31, U32, U33, U34, U35, U36, U37, U38, U39, U4, U40, U41, U42, U43, U44, U45, U46, U47, U48, U49, U5, U50, U51, U52, U53, U54, U55, U56, U57, U58, U59, U6, U60, U61, U62, U63, U64, U7, U8, U9: footprint AnodePads:anode_square_pad -> AnodePads:anode_square_pad_no_hole
