File: Design2_TwoBoardPogoPin/Board1 - Pad and Pogo Pin/Board1_Pad_PogoPin.kicad_pcb (KiCad board)
At the start: 2 copper layers, 244.9 x 299.4 mm, 150 parts, among them J1 Conn_01x01_Pin, J10 Conn_01x01_Pin, J11 Conn_01x01_Pin, J12 Conn_01x01_Pin, J13 Conn_01x01_Pin, J14 Conn_01x01_Pin, J15 Conn_01x01_Pin, J16 Conn_01x01_Pin, J17 Conn_01x01_Pin, J18 Conn_01x01_Pin, J19 Conn_01x01_Pin, J2 Conn_01x01_Pin, J20 Conn_01x01_Pin, J21 Conn_01x01_Pin, J22 Conn_01x01_Pin, J23 Conn_01x01_Pin, J24 Conn_01x01_Pin, J25 Conn_01x01_Pin, J26 Conn_01x01_Pin, J27 Conn_01x01_Pin, J28 Conn_01x01_Pin, J29 Conn_01x01_Pin, J3 Conn_01x01_Pin, J30 Conn_01x01_Pin, J31 Conn_01x01_Pin, J32 Conn_01x01_Pin, J33 Conn_01x01_Pin, J34 Conn_01x01_Pin, J35 Conn_01x01_Pin, J36 Conn_01x01_Pin, J37 Conn_01x01_Pin, J38 Conn_01x01_Pin, J39 Conn_01x01_Pin, J4 Conn_01x01_Pin, J40 Conn_01x01_Pin, J41 Conn_01x01_Pin, J42 Conn_01x01_Pin, J43 Conn_01x01_Pin, J44 Conn_01x01_Pin, J45 Conn_01x01_Pin, J46 Conn_01x01_Pin, J47 Conn_01x01_Pin, J48 Conn_01x01_Pin, J49 Conn_01x01_Pin, J5 Conn_01x01_Pin, J50 Conn_01x01_Pin, J51 Conn_01x01_Pin, J52 Conn_01x01_Pin, J53 Conn_01x01_Pin, J54 Conn_01x01_Pin, J55 Conn_01x01_Pin, J56 Conn_01x01_Pin, J57 Conn_01x01_Pin, J58 Conn_01x01_Pin, J59 Conn_01x01_Pin, J6 Conn_01x01_Pin, J60 Conn_01x01_Pin, J61 Conn_01x01_Pin, J62 Conn_01x01_Pin, J63 Conn_01x01_Pin, J64 Conn_01x01_Pin, J7 Conn_01x01_Pin, J8 Conn_01x01_Pin, J9 Conn_01x01_Pin, U1 anode_pad, U10 anode_pad, U11 anode_pad, U12 anode_pad, U13 anode_pad, U14 anode_pad, U15 anode_pad, U16 anode_pad, U17 anode_pad, U18 anode_pad, U19 anode_pad, U2 anode_pad, U20 anode_pad, U21 anode_pad, U22 anode_pad, U23 anode_pad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

Commit message: Finished two board design, waiting for review
Parts:
- added REF**: Mounting_Wuerth_WA-SMSI-M1.6_H6mm_ThreadDepth2mm_NoNPTH_977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, Mounting_Wuerth:Mounting_Wuerth_WA-SMSI-M1.6_H6mm_ThreadDepth2mm_NoNPTH_97730606330, B.Cu at (359.9, 151.6)
- added REF**10: Mounting_Wuerth_WA-SMSI-M1.6_H6mm_ThreadDepth2mm_NoNPTH_977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, Mounting_Wuerth:Mounting_Wuerth_WA-SMSI-M1.6_H6mm_ThreadDepth2mm_NoNPTH_97730606330, B.Cu at (359.9, 177.0)
- added REF**11: Mounting_Wuerth_WA-SMSI-M1.6_H6mm_ThreadDepth2mm_NoNPTH_977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, Mounting_Wuerth:Mounting_Wuerth_WA-SMSI-M1.6_H6mm_ThreadDepth2mm_NoNPTH_97730606330, B.Cu at (334.5, 177.0)
- added REF**12: Mounting_Wuerth_WA-SMSI-M1.6_H6mm_ThreadDepth2mm_NoNPTH_977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, Mounting_Wuerth:Mounting_Wuerth_WA-SMSI-M1.6_H6mm_ThreadDepth2mm_NoNPTH_97730606330, B.Cu at (309.1, 177.0)
- added REF**13: Mounting_Wuerth_WA-SMSI-M1.6_H6mm_ThreadDepth2mm_NoNPTH_977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, Mounting_Wuerth:Mounting_Wuerth_WA-SMSI-M1.6_H6mm_ThreadDepth2mm_NoNPTH_97730606330, B.Cu at (283.7, 177.0)
- added REF**14: Mounting_Wuerth_WA-SMSI-M1.6_H6mm_ThreadDepth2mm_NoNPTH_977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, Mounting_Wuerth:Mounting_Wuerth_WA-SMSI-M1.6_H6mm_ThreadDepth2mm_NoNPTH_97730606330, B.Cu at (258.3, 177.0)
- added REF**15: Mounting_Wuerth_WA-SMSI-M1.6_H6mm_ThreadDepth2mm_NoNPTH_977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, Mounting_Wuerth:Mounting_Wuerth_WA-SMSI-M1.6_H6mm_ThreadDepth2mm_NoNPTH_97730606330, B.Cu at (232.9, 177.0)
- added REF**16: Mounting_Wuerth_WA-SMSI-M1.6_H6mm_ThreadDepth2mm_NoNPTH_977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, Mounting_Wuerth:Mounting_Wuerth_WA-SMSI-M1.6_H6mm_ThreadDepth2mm_NoNPTH_97730606330, B.Cu at (207.5, 177.0)
- added REF**17: Mounting_Wuerth_WA-SMSI-M1.6_H6mm_ThreadDepth2mm_NoNPTH_977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, Mounting_Wuerth:Mounting_Wuerth_WA-SMSI-M1.6_H6mm_ThreadDepth2mm_NoNPTH_97730606330, B.Cu at (359.9, 202.4)
- added REF**18: Mounting_Wuerth_WA-SMSI-M1.6_H6mm_ThreadDepth2mm_NoNPTH_977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, Mounting_Wuerth:Mounting_Wuerth_WA-SMSI-M1.6_H6mm_ThreadDepth2mm_NoNPTH_97730606330, B.Cu at (334.5, 202.4)
- added REF**19: Mounting_Wuerth_WA-SMSI-M1.6_H6mm_ThreadDepth2mm_NoNPTH_977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, Mounting_Wuerth:Mounting_Wuerth_WA-SMSI-M1.6_H6mm_ThreadDepth2mm_NoNPTH_97730606330, B.Cu at (309.1, 202.4)
- added REF**20: Mounting_Wuerth_WA-SMSI-M1.6_H6mm_ThreadDepth2mm_NoNPTH_977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, Mounting_Wuerth:Mounting_Wuerth_WA-SMSI-M1.6_H6mm_ThreadDepth2mm_NoNPTH_97730606330, B.Cu at (283.7, 202.4)
- added REF**21: Mounting_Wuerth_WA-SMSI-M1.6_H6mm_ThreadDepth2mm_NoNPTH_977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, Mounting_Wuerth:Mounting_Wuerth_WA-SMSI-M1.6_H6mm_ThreadDepth2mm_NoNPTH_97730606330, B.Cu at (258.3, 202.4)
- added REF**22: Mounting_Wuerth_WA-SMSI-M1.6_H6mm_ThreadDepth2mm_NoNPTH_977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, Mounting_Wuerth:Mounting_Wuerth_WA-SMSI-M1.6_H6mm_ThreadDepth2mm_NoNPTH_97730606330, B.Cu at (232.9, 202.4)
- added REF**23: Mounting_Wuerth_WA-SMSI-M1.6_H6mm_ThreadDepth2mm_NoNPTH_977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, Mounting_Wuerth:Mounting_Wuerth_WA-SMSI-M1.6_H6mm_ThreadDepth2mm_NoNPTH_97730606330, B.Cu at (207.5, 202.4)
- added REF**24: Mounting_Wuerth_WA-SMSI-M1.6_H6mm_ThreadDepth2mm_NoNPTH_977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, Mounting_Wuerth:Mounting_Wuerth_WA-SMSI-M1.6_H6mm_ThreadDepth2mm_NoNPTH_97730606330, B.Cu at (359.9, 227.8)
- added REF**25: Mounting_Wuerth_WA-SMSI-M1.6_H6mm_ThreadDepth2mm_NoNPTH_977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, Mounting_Wuerth:Mounting_Wuerth_WA-SMSI-M1.6_H6mm_ThreadDepth2mm_NoNPTH_97730606330, B.Cu at (334.5, 227.8)
- added REF**26: Mounting_Wuerth_WA-SMSI-M1.6_H6mm_ThreadDepth2mm_NoNPTH_977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, Mounting_Wuerth:Mounting_Wuerth_WA-SMSI-M1.6_H6mm_ThreadDepth2mm_NoNPTH_97730606330, B.Cu at (309.1, 227.8)
- added REF**27: Mounting_Wuerth_WA-SMSI-M1.6_H6mm_ThreadDepth2mm_NoNPTH_977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, Mounting_Wuerth:Mounting_Wuerth_WA-SMSI-M1.6_H6mm_ThreadDepth2mm_NoNPTH_97730606330, B.Cu at (283.7, 227.8)
- added REF**28: Mounting_Wuerth_WA-SMSI-M1.6_H6mm_ThreadDepth2mm_NoNPTH_977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, Mounting_Wuerth:Mounting_Wuerth_WA-SMSI-M1.6_H6mm_ThreadDepth2mm_NoNPTH_97730606330, B.Cu at (258.3, 227.8)
- added REF**29: Mounting_Wuerth_WA-SMSI-M1.6_H6mm_ThreadDepth2mm_NoNPTH_977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, Mounting_Wuerth:Mounting_Wuerth_WA-SMSI-M1.6_H6mm_ThreadDepth2mm_NoNPTH_97730606330, B.Cu at (232.9, 227.8)
- added REF**30: Mounting_Wuerth_WA-SMSI-M1.6_H6mm_ThreadDepth2mm_NoNPTH_977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, Mounting_Wuerth:Mounting_Wuerth_WA-SMSI-M1.6_H6mm_ThreadDepth2mm_NoNPTH_97730606330, B.Cu at (207.5, 227.8)
- added REF**31: Mounting_Wuerth_WA-SMSI-M1.6_H6mm_ThreadDepth2mm_NoNPTH_977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, Mounting_Wuerth:Mounting_Wuerth_WA-SMSI-M1.6_H6mm_ThreadDepth2mm_NoNPTH_97730606330, B.Cu at (359.9, 253.2)
- added REF**32: Mounting_Wuerth_WA-SMSI-M1.6_H6mm_ThreadDepth2mm_NoNPTH_977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, Mounting_Wuerth:Mounting_Wuerth_WA-SMSI-M1.6_H6mm_ThreadDepth2mm_NoNPTH_97730606330, B.Cu at (334.5, 253.2)
- added REF**33: Mounting_Wuerth_WA-SMSI-M1.6_H6mm_ThreadDepth2mm_NoNPTH_977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, Mounting_Wuerth:Mounting_Wuerth_WA-SMSI-M1.6_H6mm_ThreadDepth2mm_NoNPTH_97730606330, B.Cu at (309.1, 253.2)
- added REF**34: Mounting_Wuerth_WA-SMSI-M1.6_H6mm_ThreadDepth2mm_NoNPTH_977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, Mounting_Wuerth:Mounting_Wuerth_WA-SMSI-M1.6_H6mm_ThreadDepth2mm_NoNPTH_97730606330, B.Cu at (283.7, 253.2)
- added REF**35: Mounting_Wuerth_WA-SMSI-M1.6_H6mm_ThreadDepth2mm_NoNPTH_977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, Mounting_Wuerth:Mounting_Wuerth_WA-SMSI-M1.6_H6mm_ThreadDepth2mm_NoNPTH_97730606330, B.Cu at (258.3, 253.2)
- added REF**36: Mounting_Wuerth_WA-SMSI-M1.6_H6mm_ThreadDepth2mm_NoNPTH_977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, Mounting_Wuerth:Mounting_Wuerth_WA-SMSI-M1.6_H6mm_ThreadDepth2mm_NoNPTH_97730606330, B.Cu at (232.9, 253.2)
- added REF**37: Mounting_Wuerth_WA-SMSI-M1.6_H6mm_ThreadDepth2mm_NoNPTH_977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, Mounting_Wuerth:Mounting_Wuerth_WA-SMSI-M1.6_H6mm_ThreadDepth2mm_NoNPTH_97730606330, B.Cu at (207.5, 253.2)
- added REF**38: Mounting_Wuerth_WA-SMSI-M1.6_H6mm_ThreadDepth2mm_NoNPTH_977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, Mounting_Wuerth:Mounting_Wuerth_WA-SMSI-M1.6_H6mm_ThreadDepth2mm_NoNPTH_97730606330, B.Cu at (359.9, 278.6)
- added REF**39: Mounting_Wuerth_WA-SMSI-M1.6_H6mm_ThreadDepth2mm_NoNPTH_977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, Mounting_Wuerth:Mounting_Wuerth_WA-SMSI-M1.6_H6mm_ThreadDepth2mm_NoNPTH_97730606330, B.Cu at (334.5, 278.6)
- added REF**4: Mounting_Wuerth_WA-SMSI-M1.6_H6mm_ThreadDepth2mm_NoNPTH_977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, Mounting_Wuerth:Mounting_Wuerth_WA-SMSI-M1.6_H6mm_ThreadDepth2mm_NoNPTH_97730606330, B.Cu at (334.5, 151.6)
- added REF**40: Mounting_Wuerth_WA-SMSI-M1.6_H6mm_ThreadDepth2mm_NoNPTH_977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, Mounting_Wuerth:Mounting_Wuerth_WA-SMSI-M1.6_H6mm_ThreadDepth2mm_NoNPTH_97730606330, B.Cu at (309.1, 278.6)
- added REF**41: Mounting_Wuerth_WA-SMSI-M1.6_H6mm_ThreadDepth2mm_NoNPTH_977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, Mounting_Wuerth:Mounting_Wuerth_WA-SMSI-M1.6_H6mm_ThreadDepth2mm_NoNPTH_97730606330, B.Cu at (283.7, 278.6)
- added REF**42: Mounting_Wuerth_WA-SMSI-M1.6_H6mm_ThreadDepth2mm_NoNPTH_977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, Mounting_Wuerth:Mounting_Wuerth_WA-SMSI-M1.6_H6mm_ThreadDepth2mm_NoNPTH_97730606330, B.Cu at (258.3, 278.6)
- added REF**43: Mounting_Wuerth_WA-SMSI-M1.6_H6mm_ThreadDepth2mm_NoNPTH_977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, Mounting_Wuerth:Mounting_Wuerth_WA-SMSI-M1.6_H6mm_ThreadDepth2mm_NoNPTH_97730606330, B.Cu at (232.9, 278.6)
- added REF**44: Mounting_Wuerth_WA-SMSI-M1.6_H6mm_ThreadDepth2mm_NoNPTH_977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, Mounting_Wuerth:Mounting_Wuerth_WA-SMSI-M1.6_H6mm_ThreadDepth2mm_NoNPTH_97730606330, B.Cu at (207.5, 278.6)
- added REF**45: Mounting_Wuerth_WA-SMSI-M1.6_H6mm_ThreadDepth2mm_NoNPTH_977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, Mounting_Wuerth:Mounting_Wuerth_WA-SMSI-M1.6_H6mm_ThreadDepth2mm_NoNPTH_97730606330, B.Cu at (359.9, 304.0)
- added REF**46: Mounting_Wuerth_WA-SMSI-M1.6_H6mm_ThreadDepth2mm_NoNPTH_977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, Mounting_Wuerth:Mounting_Wuerth_WA-SMSI-M1.6_H6mm_ThreadDepth2mm_NoNPTH_97730606330, B.Cu at (334.5, 304.0)
- added REF**47: Mounting_Wuerth_WA-SMSI-M1.6_H6mm_ThreadDepth2mm_NoNPTH_977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, Mounting_Wuerth:Mounting_Wuerth_WA-SMSI-M1.6_H6mm_ThreadDepth2mm_NoNPTH_97730606330, B.Cu at (309.1, 304.0)
- added REF**48: Mounting_Wuerth_WA-SMSI-M1.6_H6mm_ThreadDepth2mm_NoNPTH_977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, Mounting_Wuerth:Mounting_Wuerth_WA-SMSI-M1.6_H6mm_ThreadDepth2mm_NoNPTH_97730606330, B.Cu at (283.7, 304.0)
- added REF**49: Mounting_Wuerth_WA-SMSI-M1.6_H6mm_ThreadDepth2mm_NoNPTH_977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, Mounting_Wuerth:Mounting_Wuerth_WA-SMSI-M1.6_H6mm_ThreadDepth2mm_NoNPTH_97730606330, B.Cu at (258.3, 304.0)
- added REF**5: Mounting_Wuerth_WA-SMSI-M1.6_H6mm_ThreadDepth2mm_NoNPTH_977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, Mounting_Wuerth:Mounting_Wuerth_WA-SMSI-M1.6_H6mm_ThreadDepth2mm_NoNPTH_97730606330, B.Cu at (309.1, 151.6)
- added REF**50: Mounting_Wuerth_WA-SMSI-M1.6_H6mm_ThreadDepth2mm_NoNPTH_977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, Mounting_Wuerth:Mounting_Wuerth_WA-SMSI-M1.6_H6mm_ThreadDepth2mm_NoNPTH_97730606330, B.Cu at (232.9, 304.0)
- added REF**51: Mounting_Wuerth_WA-SMSI-M1.6_H6mm_ThreadDepth2mm_NoNPTH_977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, Mounting_Wuerth:Mounting_Wuerth_WA-SMSI-M1.6_H6mm_ThreadDepth2mm_NoNPTH_97730606330, B.Cu at (207.5, 304.0)
- added REF**6: Mounting_Wuerth_WA-SMSI-M1.6_H6mm_ThreadDepth2mm_NoNPTH_977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, Mounting_Wuerth:Mounting_Wuerth_WA-SMSI-M1.6_H6mm_ThreadDepth2mm_NoNPTH_97730606330, B.Cu at (283.7, 151.6)
- added REF**7: Mounting_Wuerth_WA-SMSI-M1.6_H6mm_ThreadDepth2mm_NoNPTH_977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, Mounting_Wuerth:Mounting_Wuerth_WA-SMSI-M1.6_H6mm_ThreadDepth2mm_NoNPTH_97730606330, B.Cu at (258.3, 151.6)
- added REF**8: Mounting_Wuerth_WA-SMSI-M1.6_H6mm_ThreadDepth2mm_NoNPTH_977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, Mounting_Wuerth:Mounting_Wuerth_WA-SMSI-M1.6_H6mm_ThreadDepth2mm_NoNPTH_97730606330, B.Cu at (232.9, 151.6)
- added REF**9: Mounting_Wuerth_WA-SMSI-M1.6_H6mm_ThreadDepth2mm_NoNPTH_977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, Mounting_Wuerth:Mounting_Wuerth_WA-SMSI-M1.6_H6mm_ThreadDepth2mm_NoNPTH_97730606330, B.Cu at (207.5, 151.6)
Routing:
- removed copper zone on F.Cu, net (none)

Commit message: May 12 update
Parts:
- REF**, REF**10, REF**11, REF**12, REF**13, REF**14, REF**15, REF**16, REF**17, REF**18, REF**19, REF**20, REF**21, REF**22, REF**23, REF**24, REF**25, REF**26, REF**27, REF**28, REF**29, REF**30, REF**31, REF**32, REF**33, REF**34, REF**35, REF**36, REF**37, REF**38, REF**39, REF**4, REF**40, REF**41, REF**42, REF**43, REF**44, REF**45, REF**46, REF**47, REF**48, REF**49, REF**5, REF**50, REF**51, REF**6, REF**7, REF**8, REF**9: value Mounting_Wuerth_WA-SMSI-M1.6_H6mm_ThreadDepth2mm_NoNPTH_97730606330 -> Standoff_mount_5.5D; footprint Mounting_Wuerth:Mounting_Wuerth_WA-SMSI-M1.6_H6mm_ThreadDepth2mm_NoNPTH_97730606330 -> AnodePads:Standoff_mount_5.5D
