File: Design2_TwoBoardPogoPin/Board2 - Housing and Samtech/Board2 - Housing and Samtech.kicad_sch (KiCad schematic)
At the start: 70 parts, among them J1 QRM8-078-05.0-L-D-A, J2 QRM8-078-05.0-L-D-A, U1 anode_pad, U10 anode_pad, U11 anode_pad, U12 anode_pad, U13 anode_pad, U14 anode_pad, U15 anode_pad, U16 anode_pad, U17 anode_pad, U18 anode_pad, U19 anode_pad, U2 anode_pad, U20 anode_pad, U21 anode_pad, U22 anode_pad, U23 anode_pad, U24 anode_pad, U25 anode_pad, U26 anode_pad, U27 anode_pad, U28 anode_pad, U29 anode_pad, U3 anode_pad, U30 anode_pad, U31 anode_pad, U32 anode_pad, U33 anode_pad, U34 anode_pad, U35 anode_pad, U36 anode_pad, U37 anode_pad, U38 anode_pad, U39 anode_pad, U4 anode_pad, U40 anode_pad, U41 anode_pad, U42 anode_pad, U43 anode_pad, U44 anode_pad, U45 anode_pad, U46 anode_pad, U47 anode_pad, U48 anode_pad, U49 anode_pad, U5 anode_pad, U50 anode_pad, U51 anode_pad, U52 anode_pad, U53 anode_pad, U54 anode_pad, U55 anode_pad, U56 anode_pad, U57 anode_pad, U58 anode_pad, U59 anode_pad, U6 anode_pad, U60 anode_pad, U61 anode_pad, U62 anode_pad, U63 anode_pad, U64 anode_pad, U7 anode_pad, U8 anode_pad, U9 anode_pad

Commit message: Finished two board design, waiting for review
Connections:
- net a2: now also J1.132; no longer J1.24
- net a3: now also J1.136; no longer J1.20
- net a4: now also J1.128; no longer J1.28
- net a5: now also J2.28; no longer J2.128
- net a6: now also J2.20; no longer J2.136
- net a7: now also J2.24; no longer J2.132
- net b1: now also J1.120; no longer J1.36
- net b2: now also J1.116; no longer J1.40
- net b3: now also J1.124; no longer J1.32
- net b4: now also J1.112; no longer J1.44
- net b5: now also J2.44; no longer J2.112
- net b6: now also J2.32; no longer J2.124
- net b7: now also J2.40; no longer J2.116
- net b8: now also J2.36; no longer J2.120
- net c1: now also J1.104; no longer J1.52
- net c2: now also J1.100; no longer J1.56
- net c3: now also J1.108; no longer J1.48
- net c4: now also J1.96; no longer J1.60
- net c5: now also J2.60; no longer J2.96
- net c6: now also J2.48; no longer J2.108
- net c7: now also J2.56; no longer J2.100
- net c8: now also J2.52; no longer J2.104
- net d1: now also J1.88; no longer J1.68
- net d2: now also J1.84; no longer J1.72
- net d3: now also J1.92; no longer J1.64
- net d4: now also J1.80; no longer J1.76
- net d5: now also J2.76; no longer J2.80
- net d6: now also J2.64; no longer J2.92
- net d7: now also J2.72; no longer J2.84
- net d8: now also J2.68; no longer J2.88
- net e1: now also J1.68; no longer J1.88
- net e2: now also J1.72; no longer J1.84
- net e3: now also J1.64; no longer J1.92
- net e4: now also J1.76; no longer J1.80
- net e5: now also J2.80; no longer J2.76
- net e6: now also J2.92; no longer J2.64
- net e7: now also J2.84; no longer J2.72
- net e8: now also J2.88; no longer J2.68
- net f1: now also J1.52; no longer J1.104
- net f2: now also J1.56; no longer J1.100
- net f3: now also J1.48; no longer J1.108
- net f4: now also J1.60; no longer J1.96
- net f5: now also J2.96; no longer J2.60
- net f6: now also J2.108; no longer J2.48
- net f7: now also J2.100; no longer J2.56
- net f8: now also J2.104; no longer J2.52
- net g1: now also J1.36; no longer J1.120
- net g2: now also J1.40; no longer J1.116
- net g3: now also J1.32; no longer J1.124
- net g4: now also J1.44; no longer J1.112
- net g5: now also J2.112; no longer J2.44
- net g6: now also J2.124; no longer J2.32
- net g7: now also J2.116; no longer J2.40
- net g8: now also J2.120; no longer J2.36
- net h2: now also J1.24; no longer J1.132
- net h3: now also J1.20; no longer J1.136
- net h4: now also J1.28; no longer J1.128
- net h5: now also J2.128; no longer J2.28
- net h6: now also J2.136; no longer J2.20
- net h7: now also J2.132; no longer J2.24
