File: Design2_TwoBoardPogoPin/Board2 - Housing and Samtech/Board2 - Housing and Samtech.kicad_pcb (KiCad board)
At the start: 2 copper layers, 244.9 x 299.4 mm, 161 parts, among them J1 QRM8-078-05.0-L-D-A, J10 Conn_01x01_Pin, J11 Conn_01x01_Pin, J12 Conn_01x01_Pin, J13 Conn_01x01_Pin, J14 Conn_01x01_Pin, J15 Conn_01x01_Pin, J16 Conn_01x01_Pin, J17 Conn_01x01_Pin, J18 Conn_01x01_Pin, J19 Conn_01x01_Pin, J2 QRM8-078-05.0-L-D-A, J20 Conn_01x01_Pin, J21 Conn_01x01_Pin, J22 Conn_01x01_Pin, J23 Conn_01x01_Pin, J24 Conn_01x01_Pin, J25 Conn_01x01_Pin, J26 Conn_01x01_Pin, J27 Conn_01x01_Pin, J28 Conn_01x01_Pin, J29 Conn_01x01_Pin, J3 Conn_01x01_Pin, J30 Conn_01x01_Pin, J31 Conn_01x01_Pin, J32 Conn_01x01_Pin, J33 Conn_01x01_Pin, J34 Conn_01x01_Pin, J35 Conn_01x01_Pin, J36 Conn_01x01_Pin, J37 Conn_01x01_Pin, J38 Conn_01x01_Pin, J39 Conn_01x01_Pin, J4 Conn_01x01_Pin, J40 Conn_01x01_Pin, J41 Conn_01x01_Pin, J42 Conn_01x01_Pin, J43 Conn_01x01_Pin, J44 Conn_01x01_Pin, J45 Conn_01x01_Pin, J46 Conn_01x01_Pin, J47 Conn_01x01_Pin, J48 Conn_01x01_Pin, J49 Conn_01x01_Pin, J5 Conn_01x01_Pin, J50 Conn_01x01_Pin, J51 Conn_01x01_Pin, J52 Conn_01x01_Pin, J53 Conn_01x01_Pin, J54 Conn_01x01_Pin, J55 Conn_01x01_Pin, J56 Conn_01x01_Pin, J57 Conn_01x01_Pin, J58 Conn_01x01_Pin, J59 Conn_01x01_Pin, J6 Conn_01x01_Pin, J60 Conn_01x01_Pin, J61 Conn_01x01_Pin, J62 Conn_01x01_Pin, J63 Conn_01x01_Pin, J64 Conn_01x01_Pin, J7 Conn_01x01_Pin, J8 Conn_01x01_Pin, J9 Conn_01x01_Pin, U1 anode_pad, U10 anode_pad, U11 anode_pad, U12 anode_pad, U13 anode_pad, U14 anode_pad, U15 anode_pad, U16 anode_pad, U17 anode_pad, U18 anode_pad, U19 anode_pad, U2 anode_pad, U20 anode_pad, U21 anode_pad, U22 anode_pad, U23 anode_pad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

Commit message: Finished two board design, waiting for review
Parts:
- removed the ? at (306.9, 330.3) (x2)
- removed the ? at (265.5, 330.3)
- removed the ? at (224.0, 330.3)
- removed the ? at (348.4, 330.3) (x2)
- removed the ? at (327.6, 330.3) (x2)
- removed the ? at (244.7, 330.3)
- removed the ? at (286.1, 330.3)
- removed J10, J11, J12, J13, J14, J15, J16, J17, J18, J19, J20, J21, J22, J23, J24, J25, J26, J27, J28, J29, J3, J30, J31, J32, J33, J34, J35, J36, J37, J38, J39, J4, J40, J41, J42, J43, J44, J45, J46, J47, J48, J49, J5, J50, J51, J52, J53, J54, J55, J56, J57, J58, J59, J6, J60, J61, J62, J63, J64, J7, J8, J9: Conn_01x01_Pin, AnodePads:PogoPinWithTail
- added ?: , , B.Cu at (327.6, 330.3)
- added ?: , , B.Cu at (306.9, 330.3)
- added ?: , , B.Cu at (348.4, 330.3)
- added REF**: MountingHole_2.5mm, MountingHole:MountingHole_2.5mm, F.Cu at (210.0, 134.1)
- added REF**10: MountingHole_2.5mm, MountingHole:MountingHole_2.5mm, F.Cu at (210.0, 159.5)
- added REF**11: MountingHole_2.5mm, MountingHole:MountingHole_2.5mm, F.Cu at (235.4, 159.5)
- added REF**12: MountingHole_2.5mm, MountingHole:MountingHole_2.5mm, F.Cu at (260.8, 159.5)
- added REF**13: MountingHole_2.5mm, MountingHole:MountingHole_2.5mm, F.Cu at (286.2, 159.5)
- added REF**14: MountingHole_2.5mm, MountingHole:MountingHole_2.5mm, F.Cu at (311.6, 159.5)
- added REF**15: MountingHole_2.5mm, MountingHole:MountingHole_2.5mm, F.Cu at (337.0, 159.5)
- added REF**16: MountingHole_2.5mm, MountingHole:MountingHole_2.5mm, F.Cu at (362.4, 159.5)
- added REF**17: MountingHole_2.5mm, MountingHole:MountingHole_2.5mm, F.Cu at (210.0, 184.9)
- added REF**18: MountingHole_2.5mm, MountingHole:MountingHole_2.5mm, F.Cu at (235.4, 184.9)
- added REF**19: MountingHole_2.5mm, MountingHole:MountingHole_2.5mm, F.Cu at (260.8, 184.9)
- added REF**20: MountingHole_2.5mm, MountingHole:MountingHole_2.5mm, F.Cu at (286.2, 184.9)
- added REF**21: MountingHole_2.5mm, MountingHole:MountingHole_2.5mm, F.Cu at (311.6, 184.9)
- added REF**22: MountingHole_2.5mm, MountingHole:MountingHole_2.5mm, F.Cu at (337.0, 184.9)
- added REF**23: MountingHole_2.5mm, MountingHole:MountingHole_2.5mm, F.Cu at (362.4, 184.9)
- added REF**24: MountingHole_2.5mm, MountingHole:MountingHole_2.5mm, F.Cu at (210.0, 210.3)
- added REF**25: MountingHole_2.5mm, MountingHole:MountingHole_2.5mm, F.Cu at (235.4, 210.3)
- added REF**26: MountingHole_2.5mm, MountingHole:MountingHole_2.5mm, F.Cu at (260.8, 210.3)
- added REF**27: MountingHole_2.5mm, MountingHole:MountingHole_2.5mm, F.Cu at (286.2, 210.3)
- added REF**28: MountingHole_2.5mm, MountingHole:MountingHole_2.5mm, F.Cu at (311.6, 210.3)
- added REF**29: MountingHole_2.5mm, MountingHole:MountingHole_2.5mm, F.Cu at (337.0, 210.3)
- added REF**30: MountingHole_2.5mm, MountingHole:MountingHole_2.5mm, F.Cu at (362.4, 210.3)
- added REF**31: MountingHole_2.5mm, MountingHole:MountingHole_2.5mm, F.Cu at (210.0, 235.7)
- added REF**32: MountingHole_2.5mm, MountingHole:MountingHole_2.5mm, F.Cu at (235.4, 235.7)
- added REF**33: MountingHole_2.5mm, MountingHole:MountingHole_2.5mm, F.Cu at (260.8, 235.7)
- added REF**34: MountingHole_2.5mm, MountingHole:MountingHole_2.5mm, F.Cu at (286.2, 235.7)
- added REF**35: MountingHole_2.5mm, MountingHole:MountingHole_2.5mm, F.Cu at (311.6, 235.7)
- added REF**36: MountingHole_2.5mm, MountingHole:MountingHole_2.5mm, F.Cu at (337.0, 235.7)
- added REF**37: MountingHole_2.5mm, MountingHole:MountingHole_2.5mm, F.Cu at (362.4, 235.7)
- added REF**38: MountingHole_2.5mm, MountingHole:MountingHole_2.5mm, F.Cu at (210.0, 261.1)
- added REF**39: MountingHole_2.5mm, MountingHole:MountingHole_2.5mm, F.Cu at (235.4, 261.1)
- added REF**4: MountingHole_2.5mm, MountingHole:MountingHole_2.5mm, F.Cu at (235.4, 134.1)
- added REF**40: MountingHole_2.5mm, MountingHole:MountingHole_2.5mm, F.Cu at (260.8, 261.1)
- added REF**41: MountingHole_2.5mm, MountingHole:MountingHole_2.5mm, F.Cu at (286.2, 261.1)
- added REF**42: MountingHole_2.5mm, MountingHole:MountingHole_2.5mm, F.Cu at (311.6, 261.1)
- added REF**43: MountingHole_2.5mm, MountingHole:MountingHole_2.5mm, F.Cu at (337.0, 261.1)
- added REF**44: MountingHole_2.5mm, MountingHole:MountingHole_2.5mm, F.Cu at (362.4, 261.1)
- added REF**45: MountingHole_2.5mm, MountingHole:MountingHole_2.5mm, F.Cu at (210.0, 286.5)
- added REF**46: MountingHole_2.5mm, MountingHole:MountingHole_2.5mm, F.Cu at (235.4, 286.5)
- added REF**47: MountingHole_2.5mm, MountingHole:MountingHole_2.5mm, F.Cu at (260.8, 286.5)
- added REF**48: MountingHole_2.5mm, MountingHole:MountingHole_2.5mm, F.Cu at (286.2, 286.5)
- added REF**49: MountingHole_2.5mm, MountingHole:MountingHole_2.5mm, F.Cu at (311.6, 286.5)
- added REF**5: MountingHole_2.5mm, MountingHole:MountingHole_2.5mm, F.Cu at (260.8, 134.1)
- added REF**50: MountingHole_2.5mm, MountingHole:MountingHole_2.5mm, F.Cu at (337.0, 286.5)
- added REF**51: MountingHole_2.5mm, MountingHole:MountingHole_2.5mm, F.Cu at (362.4, 286.5)
- added REF**6: MountingHole_2.5mm, MountingHole:MountingHole_2.5mm, F.Cu at (286.2, 134.1)
- added REF**7: MountingHole_2.5mm, MountingHole:MountingHole_2.5mm, F.Cu at (311.6, 134.1)
- added REF**8: MountingHole_2.5mm, MountingHole:MountingHole_2.5mm, F.Cu at (337.0, 134.1)
- added REF**9: MountingHole_2.5mm, MountingHole:MountingHole_2.5mm, F.Cu at (362.4, 134.1)
- moved J1 12.2 mm to (285.8, 68.6), turned to 180 degrees
- moved J2 12.2 mm to (286.5, 352.1), turned to 0 degrees
Connections:
- J1 pad 100: /f2 -> /c2
- J1 pad 104: /f1 -> /c1
- J1 pad 108: /f3 -> /c3
- J1 pad 112: /g4 -> /b4
- J1 pad 116: /g2 -> /b2
- J1 pad 120: /g1 -> /b1
- J1 pad 124: /g3 -> /b3
- J1 pad 128: /h4 -> /a4
- J1 pad 132: /h2 -> /a2
- J1 pad 136: /h3 -> /a3
- J1 pad 20: /a3 -> /h3
- J1 pad 24: /a2 -> /h2
- J1 pad 28: /a4 -> /h4
- J1 pad 32: /b3 -> /g3
- J1 pad 36: /b1 -> /g1
- J1 pad 40: /b2 -> /g2
- J1 pad 44: /b4 -> /g4
- J1 pad 48: /c3 -> /f3
- J1 pad 52: /c1 -> /f1
- J1 pad 56: /c2 -> /f2
- J1 pad 60: /c4 -> /f4
- J1 pad 64: /d3 -> /e3
- J1 pad 68: /d1 -> /e1
- J1 pad 72: /d2 -> /e2
- J1 pad 76: /d4 -> /e4
- J1 pad 80: /e4 -> /d4
- J1 pad 84: /e2 -> /d2
- J1 pad 88: /e1 -> /d1
- J1 pad 92: /e3 -> /d3
- J1 pad 96: /f4 -> /c4
- J2 pad 100: /c7 -> /f7
- J2 pad 104: /c8 -> /f8
- J2 pad 108: /c6 -> /f6
- J2 pad 112: /b5 -> /g5
- J2 pad 116: /b7 -> /g7
- J2 pad 120: /b8 -> /g8
- J2 pad 124: /b6 -> /g6
- J2 pad 128: /a5 -> /h5
- J2 pad 132: /a7 -> /h7
- J2 pad 136: /a6 -> /h6
- J2 pad 20: /h6 -> /a6
- J2 pad 24: /h7 -> /a7
- J2 pad 28: /h5 -> /a5
- J2 pad 32: /g6 -> /b6
- J2 pad 36: /g8 -> /b8
- J2 pad 40: /g7 -> /b7
- J2 pad 44: /g5 -> /b5
- J2 pad 48: /f6 -> /c6
- J2 pad 52: /f8 -> /c8
- J2 pad 56: /f7 -> /c7
- J2 pad 60: /f5 -> /c5
- J2 pad 64: /e6 -> /d6
- J2 pad 68: /e8 -> /d8
- J2 pad 72: /e7 -> /d7
- J2 pad 76: /e5 -> /d5
- J2 pad 80: /d5 -> /e5
- J2 pad 84: /d7 -> /e7
- J2 pad 88: /d8 -> /e8
- J2 pad 92: /d6 -> /e6
- J2 pad 96: /c5 -> /f5
Routing:
- net /d5: track 140.0 -> 173.4 mm, vias 2 -> 0
- net /e5: track 145.3 -> 172.9 mm, vias 2 -> 0
- net GND: track 732.7 -> 706.3 mm
- net /a8: track 39.5 -> 58.7 mm
- net /b3: track 153.6 -> 135.3 mm, vias 2 -> 0
- net /g6: track 153.5 -> 135.3 mm, vias 2 -> 0
- net /d8: track 57.3 -> 74.3 mm, vias 2 -> 0
- net /h6: track 134.8 -> 151.8 mm
- net /e8: track 59.1 -> 74.9 mm, vias 2 -> 0
- net /g5: track 166.3 -> 153.8 mm, vias 2 -> 0
- net /d7: track 89.6 -> 100.0 mm, vias 2 -> 0
- net /b4: track 163.5 -> 153.8 mm, vias 2 -> 0
- net /g8: track 89.8 -> 80.5 mm, vias 2 -> 0
- net /e7: track 85.4 -> 94.1 mm, vias 2 -> 0
- net /g3: track 142.6 -> 135.2 mm, vias 2 -> 0
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Other:
- board outline removed

Commit message: update step files
Other:
- board outline added: 244.9 x 299.4 mm
Changed lines of the file:
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@@
     )
   )
+  (gr_poly
+    (pts
+      (xy 164.266679 61.61255)
+      (xy 409.173479 61.61255)
+      (xy 409.173479 360.97695)
+      (xy 164.266679 360.97695)
+    )
+    (stroke (width 0.2) (type solid)) (fill none) (layer "Edge.Cuts"))
   (via (at 184.5564 159.5374) (size 0.8) (drill 0.4) (layers "F.Cu" "B.Cu") (net 0))
   (via (at 387.7564 261.1374) (size 0.8) (drill 0.4) (layers "F.Cu" "B.Cu") (net 0))

Commit message: May 12 update
Parts:
- REF**, REF**10, REF**11, REF**12, REF**13, REF**14, REF**15, REF**16, REF**17, REF**18, REF**19, REF**20, REF**21, REF**22, REF**23, REF**24, REF**25, REF**26, REF**27, REF**28, REF**29, REF**30, REF**31, REF**32, REF**33, REF**34, REF**35, REF**36, REF**37, REF**38, REF**39, REF**4, REF**40, REF**41, REF**42, REF**43, REF**44, REF**45, REF**46, REF**47, REF**48, REF**49, REF**5, REF**50, REF**51, REF**6, REF**7, REF**8, REF**9: value MountingHole_2.5mm -> MountingHole_3.2mm_M3_ISO14580; footprint MountingHole:MountingHole_2.5mm -> MountingHole:MountingHole_3.2mm_M3_ISO14580
- U1, U10, U11, U12, U13, U14, U15, U16, U17, U18, U19, U2, U20, U21, U22, U23, U24, U25, U26, U27, U28, U29, U3, U30, U31, U32, U33, U34, U35, U36, U37, U38, U39, U4, U40, U41, U42, U43, U44, U45, U46, U47, U48, U49, U5, U50, U51, U52, U53, U54, U55, U56, U57, U58, U59, U6, U60, U61, U62, U63, U64, U7, U8, U9: footprint Connector_Pin:Pin_D0.7mm_L6.5mm_W1.8mm_FlatFork -> AnodePads:PogoPinWithTail
Routing:
- net GND: track 706.3 -> 883.0 mm, vias 0 -> 838
- net /d7: track 100.0 -> 87.8 mm
- net /e7: track 94.1 -> 89.7 mm
- net /d2: track 85.5 -> 81.1 mm
- net /b7: track 108.8 -> 105.2 mm
- net /h7: track 125.1 -> 121.6 mm
- net /h2: track 125.1 -> 121.5 mm
- net /g7: track 108.9 -> 105.3 mm
- net /b2: track 108.9 -> 105.3 mm
- net /g2: track 108.8 -> 105.2 mm
- net /c7: track 94.5 -> 90.9 mm
- net /a7: track 125.1 -> 121.5 mm
- net /f7: track 92.6 -> 89.0 mm
- net /e2: track 84.7 -> 81.1 mm
- net /c2: track 92.6 -> 89.0 mm
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- added copper zone on In1.Cu, net GND
- added copper zone on In2.Cu, net GND
Other:
- copper layers 2 -> 4
